File: PlasmaTransformer.kicad_sch (KiCad schematic)
At the start: 38 parts, among them J1 Barrel_Jack_MountingPin, J10 Screw_Terminal_01x01, J11 Screw_Terminal_01x01, J12 Screw_Terminal_01x01, J2 Conn_01x02_Pin, J3 Conn_Coaxial, J5 Conn_Coaxial, J6 Screw_Terminal_01x01, J7 Screw_Terminal_01x01, J8 AudioJack3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

Commit message: layout complete, commit before resync
Connections:
- net at J7.1 (Pin_1), JP1.2 (B), JP2.2 (B)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: now also H1.1
- net at J12.1 (Pin_1), J6.1 (Pin_1): no longer H1.1
Other:
- moved on the sheet: H1
Changed lines of the file:
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@@
+	)
+	(junction
+		(at 203.2 91.44)
+		(diameter 0)
+		(color 0 0 0 0)
 	)
 	(junction
@@
 	)
 	(junction
-		(at 257.81 91.44)
-		(diameter 0)
-		(color 0 0 0 0)
-	)
-	(junction
 		(at 177.8 82.55)
 		(diameter 0)
@@
 	(wire
 		(pts
-			(xy 264.16 91.44) (xy 257.81 91.44)
-		)
-		(stroke
-			(width 0)
-			(type default)
-		)
-	)
-	(wire
-		(pts
 			(xy 257.81 91.44) (xy 232.41 91.44)
 		)
@@
 	(wire
 		(pts
-			(xy 195.58 91.44) (xy 222.25 91.44)
+			(xy 195.58 91.44) (xy 203.2 91.44)
 		)
 		(stroke
@@
 	(wire
 		(pts
+			(xy 203.2 91.44) (xy 222.25 91.44)
+		)
+		(stroke
+			(width 0)
+			(type default)
+		)
+	)
+	(wire
+		(pts
 			(xy 177.8 82.55) (xy 177.8 91.44)
 		)
@@
 		(pts
 			(xy 71.12 59.69) (xy 82.55 59.69)
-		)
-		(stroke
-			(width 0)
-			(type default)
-		)
-	)
-	(wire
-		(pts
-			(xy 264.16 91.44) (xy 264.16 88.9)
 		)
 		(stroke
@@
 	(symbol
 		(lib_id "Mechanical:MountingHole_Pad")
-		(at 264.16 86.36 0)
+		(at 203.2 88.9 0)
 		(unit 1)
 		(exclude_from_sim no)
@@
 		(fields_autoplaced yes)
 		(property "Reference" "H1"
-			(at 266.7 83.8199 0)
+			(at 205.74 86.3599 0)
 			(effects
 				(font
@@
 		)
 		(property "Value" "MountingHole_Pad"
-			(at 266.7 86.3599 0)
+			(at 205.74 88.8999 0)
 			(effects
 				(font
@@
 		)
 		(property "Footprint" "MountingHole:MountingHole_5.3mm_M5_Pad"
-			(at 264.16 86.36 0)
+			(at 203.2 88.9 0)
 			(effects
 				(font
@@
 		)
 		(property "Datasheet" "~"
-			(at 264.16 86.36 0)
+			(at 203.2 88.9 0)
 			(effects
 				(font
@@
 		)
 		(property "Description" "Mounting Hole with connection"
-			(at 264.16 86.36 0)
-			(effects
-				(font
+			(at 203.2 88.9 0)
+			(effects
+				(font

Commit message: final edits, silkscreens, generate Rev 1 manufacturing files
Parts:
- added D3: LED, LED_SMD:LED_1206_3216Metric, symbol Device:LED
- added L1: PCB Coil, Library:FEEDBACK_COIL_B, symbol Device:L
- added R1, R10, R11, R12: 1k, Resistor_SMD:R_1812_4532Metric, symbol Device:R
- added R13: 680, Resistor_SMD:R_0805_2012Metric, symbol Device:R
Connections:
- net at C7.1, J10.1 (Pin_1), J11.1 (Pin_1)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: now also R1.1
- net at J12.1 (Pin_1), J6.1 (Pin_1): now also R12.2
- new net: R11.2, R12.1
- new net: R10.2, R11.1
- new net: R1.2, R10.1
- new net: D3.1 (K), L1.1
- new net: D3.2 (A), R13.2
- new net: L1.2, R13.1
Other:
- note added: "FEEDBACK SENSOR DESIGN BY SKY-GUIDED"

Commit message: adding BOM files and 3D design for coil support and fan shroud for 130cm globe
Parts:
- D3: MPN (none) -> 150120AS75000; Manufacturer (none) -> Wurth
- H1, H2, HS1: now not fitted
- J8: MPN (none) -> SJ-3523-SMT-TR; Manufacturer (none) -> CUI
- L1: now not fitted; now left out of the parts list
- R1, R10, R11, R12: value 1k -> 100k; MPN (none) -> ERJ-12NF1003U; Manufacturer (none) -> Panasonic
- R13: MPN (none) -> RC0805FR-07680RL; Manufacturer (none) -> Yageo
- R2, R5: MPN (none) -> RC0805FR-071KL; Manufacturer (none) -> Yageo
- R3: MPN (none) -> RC0805FR-073KL; Manufacturer (none) -> Yageo
- R4: MPN (none) -> RC0805FR-071K8L; Manufacturer (none) -> Yageo
- R6: MPN (none) -> RC0805JR-070RL; Manufacturer (none) -> Yageo
- R7, R8, R9: value 50 -> 49.9; MPN (none) -> RC0805FR-0749R9L; Manufacturer (none) -> Yageo
