File: E-Field Igniter Daughterboard/E-Field Igniter Daughterboard.kicad_pcb (KiCad board)
At the start: 2 copper layers, 74.5 x 20 mm, 21 parts, among them J1 Conn_01x02_Pin, J2 Conn_01x02_Pin, J3 Xe Strike, T1 PA0367A 1:12, T2 ZS 1052-S HT(H), U1 LT3468, U2 L7812CD2T-TR

Commit message: part selection and bom
Parts:
- R3: footprint Resistor_SMD:R_0603_1608Metric -> Resistor_SMD:R_0805_2012Metric
