File: Plasma Transformer PCB/PCB-PlasmaTransformer-RF-Node-Igniter/PlasmaTransformer-RF-Node-Igniter.kicad_pcb (KiCad board)
At the start: 2 copper layers, 90 x 90 mm, 66 parts, among them J1 Barrel_Jack_MountingPin, J11 Screw_Terminal_01x01, J12 Screw_Terminal_01x01, J2 Conn_01x02_Pin, J3 Conn_Coaxial, J4 Conn_02x04_Odd_Even, J5 Conn_Coaxial, J8 AudioJack3, M1 Fan, Q1 Q_NMOS_Depletion_GDS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

Commit message: fixced clearances and generated gerbers
Parts:
- moved C22 2.00 mm to (66.0, 134.2)
- moved C23 2.00 mm to (66.0, 139.2)
- moved C14 0.50 mm to (62.5, 126.2)
- moved C15 0.50 mm to (62.5, 131.2)
- moved D5 0.40 mm to (81.5, 136.5)
- moved D6 0.40 mm to (81.5, 142.2)
- moved D7 0.40 mm to (74.0, 133.8)
- moved D8 0.40 mm to (74.0, 139.2)
Routing:
- net Net-(D5-A): track 13.3 -> 19.5 mm
- net Net-(D6-A): track 60.6 -> 55.4 mm
- net Net-(D6-K): track 188.8 -> 192.9 mm
- net Net-(D5-K): track 55.2 -> 51.4 mm
- net Net-(C15-Pad2): track 5.00 -> 3.50 mm

Commit message: layout updates for Rev 3B > Rev 4: gate selector caps, SMD footprint for trigger coil, silkscreen updates
Parts:
- removed JP1, JP2, JP3, JP4: Jumper_2_Open, Connector_PinHeader_2.54mm:PinHeader_1x02_P2.54mm_Vertical
- removed R1: 0.05, Resistor_SMD:R_2512_6332Metric
- added J6: Conn_02x04_Odd_Even, Connector_PinHeader_2.54mm:PinHeader_2x04_P2.54mm_Vertical, F.Cu at (73.7, 104.7)
- D5, D6, D7, D8: value D_Schottky -> D
- moved R6 18.0 mm to (88.5, 102.5)
- moved C3 2.00 mm to (69.5, 94.2)
- moved C4 2.00 mm to (75.0, 94.2)
- moved C5 2.00 mm to (80.5, 94.2)
- moved C6 2.00 mm to (86.0, 94.2)
- moved TP1 1.61 mm to (130.9, 142.9)
Connections:
- J1 pad 2: /GND-IN -> GND
Routing:
- net Net-(D6-K): track 192.9 -> 164.7 mm
- net /GATE: track 76.1 -> 82.2 mm
- net /DRAIN: track 161.6 -> 164.1 mm
- net GND: track 364.5 -> 366.5 mm
- net Net-(J6-Pin_8): track 5.95 -> 7.80 mm
- net Net-(J6-Pin_2): track 5.95 -> 7.60 mm
- net Net-(T2-AA): track 15.2 -> 16.1 mm
- net Net-(J6-Pin_6): track 5.95 -> 6.57 mm
- added copper zone on F.Cu, net GND
- removed copper zone on F.Cu, net /GND-IN
Other:
- board text added: "IGNITER DESIGN BY @LTWIN8"

Commit message: 13cm V2 design WIP, updates to Rev 4 PCB
Parts:
- added T1: BO-02, ALibrary:BO-02, F.Cu at (127.2, 136.8)
- added TP2: Choke, Connector_Wire:SolderWire-1sqmm_1x01_D1.4mm_OD2.7mm, F.Cu at (142.5, 95.0)
- added TP3: Choke, Connector_Wire:SolderWire-1sqmm_1x01_D1.4mm_OD2.7mm, F.Cu at (142.5, 133.0)
- L2: value 9.2uH -> 30uH; footprint Inductor_SMD:L_APV_APH1770 -> ALibrary:B82559B_TDK
- moved L2 0.50 mm to (135.0, 121.5), turned to 0 degrees
Routing:
- net Net-(D6-A): track 55.4 -> 70.2 mm, vias 0 -> 2
- net GND: track 366.5 -> 354.3 mm, vias 11 -> 8
- net /DRAIN: track 164.1 -> 175.2 mm
- net Net-(J2-Pin_1): track 123.4 -> 128.0 mm
- net Net-(T1-Primary): track 16.1 -> 19.9 mm
- net Net-(T1-Secondary): track 3.90 -> 6.06 mm
Other:
- board text added: "REV 4 JULY 2025 E. CHIU"
- board text removed: "REV 3B JULY 2025 E. CHIU"
