File: Plasma Transformer PCB/PlasmaTransformer.kicad_sch (KiCad schematic)
At the start: 97 parts, among them J1 Barrel_Jack_MountingPin, J10 Conn_01x01_Socket, J11 Screw_Terminal_01x01, J12 Screw_Terminal_01x01, J13 Conn_01x01_Socket, J14 Conn_01x01_Socket, J15 Conn_01x01_Socket, J16 Conn_01x01_Socket, J17 Conn_01x01_Socket, J18 Conn_01x01_Socket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

Commit message: fab fixes, soldermask defined pad for SOT-23-8
Parts:
- R12: footprint (none) -> Resistor_SMD:R_0805_2012Metric; MPN (none) -> RC0805FR-0710KL; Tolerance (none) -> 1%
- U2: footprint Package_TO_SOT_SMD:SOT-23-8 -> ALibrary:SOT-23-8-Soldermask-Defined
Changed lines of the file:
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@@
 			)
 		)
-		(property "Footprint" "Package_TO_SOT_SMD:SOT-23-8"
+		(property "Footprint" "ALibrary:SOT-23-8-Soldermask-Defined"
 			(at 114.3 123.19 0)
 			(effects
@@
 			)
 		)
-		(property "Footprint" "Package_TO_SOT_SMD:SOT-23-8"
+		(property "Footprint" "ALibrary:SOT-23-8-Soldermask-Defined"
 			(at 86.36 125.73 0)
 			(effects
@@
 			)
 		)
-		(property "Footprint" ""
+		(property "Footprint" "Resistor_SMD:R_0805_2012Metric"
 			(at 87.63 135.128 90)
 			(effects
@@
 			)
 		)
+		(property "Tolerance" "1%"
+			(at 87.63 133.35 90)
+			(effects
+				(font
+					(size 1.27 1.27)
+				)
+				(hide yes)
+			)
+		)
+		(property "MPN" "RC0805FR-0710KL"
+			(at 87.63 133.35 90)
+			(effects
+				(font
+					(size 1.27 1.27)
+				)
+				(hide yes)
+			)
+		)
 		(pin "2"
 		)
@@
 			)
 		)
-		(property "Footprint" "Package_TO_SOT_SMD:SOT-23-8"
+		(property "Footprint" "ALibrary:SOT-23-8-Soldermask-Defined"
 			(at 35.56 125.73 0)
 			(effects
