File: Plasma Transformer PCB/PlasmaTransformer.kicad_sch (KiCad schematic)
At the start: 86 parts, among them J1 Barrel_Jack_MountingPin, J10 Conn_01x01_Socket, J11 Screw_Terminal_01x01, J12 Screw_Terminal_01x01, J13 Conn_01x01_Socket, J14 Conn_01x01_Socket, J15 Conn_01x01_Socket, J16 Conn_01x01_Socket, J17 Conn_01x01_Socket, J18 Conn_01x01_Socket, J19 Conn_01x01_Socket, J2 Conn_01x02_Pin, J20 Conn_01x01_Socket, J21 Conn_01x01_Socket, J3 Conn_Coaxial, J4 Conn_02x04_Odd_Even, J5 Conn_Coaxial, J6 Conn_02x04_Odd_Even, J7 Conn_01x01_Socket, J8 AudioJack3, J9 Conn_01x01_Socket, M1 Fan, Q1 Q_NMOS_Depletion_GDS, SW1 SW_SPDT, T1 BO-02, T2 ZS 1052-S HT(H), U1 LMR51610YDBVR

Commit message: updated hole size for capacitor press fit sockets
Parts:
- J10, J13, J14, J15, J16, J17, J18, J19, J20, J21, J7, J9: footprint ALibrary:H8501-05 -> AFootprints:H8501-05
Changed lines of the file:
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@@
 			)
 		)
-		(property "Footprint" "ALibrary:H8501-05"
+		(property "Footprint" "AFootprints:H8501-05"
 			(at 240.03 69.85 0)
 			(effects
@@
 			)
 		)
-		(property "Footprint" "ALibrary:H8501-05"
+		(property "Footprint" "AFootprints:H8501-05"
 			(at 233.68 69.85 0)
 			(effects
@@
 			)
 		)
-		(property "Footprint" "ALibrary:H8501-05"
+		(property "Footprint" "AFootprints:H8501-05"
 			(at 220.98 69.85 0)
 			(effects
@@
 			)
 		)
-		(property "Footprint" "ALibrary:H8501-05"
+		(property "Footprint" "AFootprints:H8501-05"
 			(at 233.68 64.77 0)
 			(effects
@@
 			)
 		)
-		(property "Footprint" "ALibrary:H8501-05"
+		(property "Footprint" "AFootprints:H8501-05"
 			(at 220.98 64.77 0)
 			(effects
@@
 			)
 		)
-		(property "Footprint" "ALibrary:H8501-05"
+		(property "Footprint" "AFootprints:H8501-05"
 			(at 252.73 64.77 0)
 			(effects
@@
 			)
 		)
-		(property "Footprint" "ALibrary:H8501-05"
+		(property "Footprint" "AFootprints:H8501-05"
 			(at 240.03 64.77 0)
 			(effects
@@
 			)
 		)
-		(property "Footprint" "ALibrary:H8501-05"
+		(property "Footprint" "AFootprints:H8501-05"
 			(at 227.33 69.85 0)
 			(effects
@@
 			)
 		)
-		(property "Footprint" "ALibrary:H8501-05"
+		(property "Footprint" "AFootprints:H8501-05"
 			(at 246.38 69.85 0)
 			(effects
@@
 			)
 		)
-		(property "Footprint" "ALibrary:H8501-05"
+		(property "Footprint" "AFootprints:H8501-05"
 			(at 246.38 64.77 0)
 			(effects
@@
 			)
 		)
-		(property "Footprint" "ALibrary:H8501-05"
+		(property "Footprint" "AFootprints:H8501-05"
 			(at 252.73 69.85 0)
 			(effects
@@
 			)
 		)
-		(property "Footprint" "ALibrary:H8501-05"
+		(property "Footprint" "AFootprints:H8501-05"
 			(at 227.33 64.77 0)
 			(effects
