File: Plasma Transformer PCB/PlasmaTransformer.kicad_sch (KiCad schematic)
At the start: 97 parts, among them J1 Barrel_Jack_MountingPin, J10 Conn_01x01_Socket, J11 Screw_Terminal_01x01, J12 Screw_Terminal_01x01, J13 Conn_01x01_Socket, J14 Conn_01x01_Socket, J15 Conn_01x01_Socket, J16 Conn_01x01_Socket, J17 Conn_01x01_Socket, J18 Conn_01x01_Socket, J19 Conn_01x01_Socket, J2 Conn_01x02_Pin, J20 Conn_01x01_Socket, J21 Conn_01x01_Socket, J3 Conn_Coaxial, J4 Conn_02x04_Odd_Even, J5 Conn_Coaxial, J6 Conn_02x04_Odd_Even, J7 Conn_01x01_Socket, J8 AudioJack3, J9 Conn_01x01_Socket, M1 Fan, Q1 Q_NMOS_Depletion_GDS, SW1 SW_SPDT, T1 BO-02, T2 ZS 1052-S HT(H), U1 LMR51610YDBVR, U2 TLV9302IDDFR

Commit message: manufacturing cleanup
Parts:
- U2: value TLV9302IDDFR -> TLV9302IDR; footprint ALibrary:SOT-23-8-Soldermask-Defined -> Package_SO:SOIC-8_3.9x4.9mm_P1.27mm; MPN TLV9302IDDFR -> TLV9302IDR
Changed lines of the file:
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@@
 			)
 		)
-		(property "Value" "TLV9302IDDFR"
+		(property "Value" "TLV9302IDR"
 			(at 119.126 118.11 0)
 			(effects
@@
 			)
 		)
-		(property "Footprint" "ALibrary:SOT-23-8-Soldermask-Defined"
+		(property "Footprint" "Package_SO:SOIC-8_3.9x4.9mm_P1.27mm"
 			(at 114.3 123.19 0)
 			(effects
@@
 			)
 		)
-		(property "MPN" "TLV9302IDDFR"
+		(property "MPN" "TLV9302IDR"
 			(at 114.3 123.19 0)
 			(effects
@@
 			)
 		)
-		(property "Value" "TLV9302IDDFR"
+		(property "Value" "TLV9302IDR"
 			(at 93.218 120.904 0)
 			(effects
@@
 			)
 		)
-		(property "Footprint" "ALibrary:SOT-23-8-Soldermask-Defined"
+		(property "Footprint" "Package_SO:SOIC-8_3.9x4.9mm_P1.27mm"
 			(at 86.36 125.73 0)
 			(effects
@@
 			)
 		)
-		(property "MPN" "TLV9302IDDFR"
+		(property "MPN" "TLV9302IDR"
 			(at 86.36 125.73 0)
 			(effects
@@
 			)
 		)
-		(property "Value" "TLV9302IDDFR"
+		(property "Value" "TLV9302IDR"
 			(at 17.018 126.746 0)
 			(effects
@@
 			)
 		)
-		(property "Footprint" "ALibrary:SOT-23-8-Soldermask-Defined"
+		(property "Footprint" "Package_SO:SOIC-8_3.9x4.9mm_P1.27mm"
 			(at 35.56 125.73 0)
 			(effects
@@
 			)
 		)
-		(property "MPN" "TLV9302IDDFR"
+		(property "MPN" "TLV9302IDR"
 			(at 35.56 125.73 0)
 			(effects

Commit message: updated hole size for press-fit capacitor sockets
Parts:
- C2: footprint ALibrary:CP_Elec_16x17.5_FK_Series -> AFootprints:CP_Elec_16x17.5_FK_Series
- J10, J13, J14, J15, J16, J17, J18, J19, J20, J21, J7, J9: footprint ALibrary:H8501-05 -> AFootprints:H8501-05
- J11, J12: footprint ALibrary:CONN_2604-3101_WAG -> AFootprints:CONN_2604-3101_WAG
- J3, J5: footprint ALibrary:SMA_Amphenol_901-144_Vertical -> AFootprints:SMA_Amphenol_901-144_Vertical
- J8: footprint ALibrary:Jack_3.5mm_CUI_SJ-3523-SMT_Horizontal -> AFootprints:Jack_3.5mm_CUI_SJ-3523-SMT_Horizontal
- L2: footprint ALibrary:B82559B_TDK -> AFootprints:B82559B_TDK
- L3: footprint ALibrary:L_Pana_PCC-KVP_5.5x5mm -> AFootprints:L_Pana_PCC-KVP_5.5x5mm
- M1: footprint Library:FAN AXIAL 92X25.4MM -> AFootprints:FAN AXIAL 92X25.4MM
- RV1: footprint ALibrary:Bourns-Potentiometer-PTD902-2 -> AFootprints:Bourns-Potentiometer-PTD902-2
- SW1: footprint ALibrary:CKSW-E101J1AV2QE2 -> AFootprints:CKSW-E101J1AV2QE2
- T1: footprint ALibrary:BO-02 -> AFootprints:BO-02
- T2: footprint ALibrary:ZS 1052-S HT(H) -> AFootprints:ZS 1052-S HT(H)
Changed lines of the file:
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@@
 			)
 		)
-		(property "Footprint" "ALibrary:Bourns-Potentiometer-PTD902-2"
+		(property "Footprint" "AFootprints:Bourns-Potentiometer-PTD902-2"
 			(at 127 74.93 0)
 			(effects
@@
 			)
 		)
-		(property "Footprint" "ALibrary:L_Pana_PCC-KVP_5.5x5mm"
+		(property "Footprint" "AFootprints:L_Pana_PCC-KVP_5.5x5mm"
 			(at 71.12 71.12 0)
 			(effects
@@
 			)
 		)
-		(property "Footprint" "ALibrary:BO-02"
+		(property "Footprint" "AFootprints:BO-02"
 			(at 187.706 140.462 0)
 			(effects
@@
 			)
 		)
-		(property "Footprint" "ALibrary:H8501-05"
+		(property "Footprint" "AFootprints:H8501-05"
 			(at 240.03 69.85 0)
 			(effects
@@
 			)
 		)
-		(property "Footprint" "ALibrary:H8501-05"
+		(property "Footprint" "AFootprints:H8501-05"
 			(at 233.68 69.85 0)
 			(effects
@@
 			)
 		)
-		(property "Footprint" "ALibrary:ZS 1052-S HT(H)"
+		(property "Footprint" "AFootprints:ZS 1052-S HT(H)"
 			(at 214.63 140.97 0)
 			(effects
@@
 			)
 		)
-		(property "Footprint" "ALibrary:SMA_Amphenol_901-144_Vertical"
+		(property "Footprint" "AFootprints:SMA_Amphenol_901-144_Vertical"
 			(at 179.07 81.28 0)
 			(effects
@@
 			)
 		)
-		(property "Footprint" "ALibrary:SMA_Amphenol_901-144_Vertical"
+		(property "Footprint" "AFootprints:SMA_Amphenol_901-144_Vertical"
 			(at 210.82 43.18 0)
 			(effects
@@
 			)
 		)
-		(property "Footprint" "ALibrary:Jack_3.5mm_CUI_SJ-3523-SMT_Horizontal"
+		(property "Footprint" "AFootprints:Jack_3.5mm_CUI_SJ-3523-SMT_Horizontal"
 			(at 171.45 99.06 0)
 			(effects
@@
 			)
 		)
-		(property "Footprint" "ALibrary:H8501-05"
+		(property "Footprint" "AFootprints:H8501-05"
 			(at 220.98 69.85 0)
 			(effects
@@
 			)
 		)
-		(property "Footprint" "ALibrary:H8501-05"
+		(property "Footprint" "AFootprints:H8501-05"
 			(at 233.68 64.77 0)
 			(effects
@@
 			)
 		)
-		(property "Footprint" "ALibrary:H8501-05"
+		(property "Footprint" "AFootprints:H8501-05"
 			(at 220.98 64.77 0)
 			(effects
@@
 			)
 		)
-		(property "Footprint" "Library:FAN AXIAL 92X25.4MM"
+		(property "Footprint" "AFootprints:FAN AXIAL 92X25.4MM"
 			(at 20.32 186.436 0)
 			(effects
@@
 			)
 		)
-		(property "Footprint" "ALibrary:H8501-05"
+		(property "Footprint" "AFootprints:H8501-05"
 			(at 252.73 64.77 0)
 			(effects
@@
 			)
 		)
-		(property "Footprint" "ALibrary:H8501-05"
+		(property "Footprint" "AFootprints:H8501-05"
 			(at 240.03 64.77 0)
 			(effects
@@
 			)
 		)
-		(property "Footprint" "ALibrary:CKSW-E101J1AV2QE2"
+		(property "Footprint" "AFootprints:CKSW-E101J1AV2QE2"
 			(at 52.07 38.1 0)
 			(effects
@@
 			)
 		)
-		(property "Footprint" "ALibrary:H8501-05"
+		(property "Footprint" "AFootprints:H8501-05"
 			(at 227.33 69.85 0)
 			(effects
@@
 			)
 		)
-		(property "Footprint" "ALibrary:H8501-05"
+		(property "Footprint" "AFootprints:H8501-05"
 			(at 246.38 69.85 0)
 			(effects
@@
 			)
 		)
-		(property "Footprint" "ALibrary:B82559B_TDK"
+		(property "Footprint" "AFootprints:B82559B_TDK"
 			(at 115.57 38.1 0)
 			(effects
@@
 			)
 		)
-		(property "Footprint" "ALibrary:CP_Elec_16x17.5_FK_Series"
+		(property "Footprint" "AFootprints:CP_Elec_16x17.5_FK_Series"
 			(at 66.04 41.91 0)
 			(effects
@@
 			)
 		)
-		(property "Footprint" "ALibrary:H8501-05"
+		(property "Footprint" "AFootprints:H8501-05"
 			(at 246.38 64.77 0)
 			(effects
@@
 			)
 		)
-		(property "Footprint" "ALibrary:CONN_2604-3101_WAG"
+		(property "Footprint" "AFootprints:CONN_2604-3101_WAG"
 			(at 269.24 33.02 0)
 			(effects
@@
 			)
 		)
-		(property "Footprint" "ALibrary:H8501-05"
+		(property "Footprint" "AFootprints:H8501-05"
 			(at 252.73 69.85 0)
 			(effects
@@
 			)
 		)
-		(property "Footprint" "ALibrary:CONN_2604-3101_WAG"
+		(property "Footprint" "AFootprints:CONN_2604-3101_WAG"
 			(at 269.24 48.26 0)
 			(effects
@@
 			)
 		)
-		(property "Footprint" "ALibrary:H8501-05"
+		(property "Footprint" "AFootprints:H8501-05"
 			(at 227.33 64.77 0)
 			(effects
